File: PCB/BLDC_motor_driver/BLDC_motor_driver.kicad_pcb (KiCad board)
At the start: 4 copper layers, 100 x 100 mm, 28 parts, among them J1 Current Sensing, J2 CAN H/L, J3 PWR, J4 Conn_01x04_Socket, Q8 CSD18533Q5A, Q9 CSD18533Q5A, U1 INA240A2D, U10 AS5048A, U11 AMS1117-3.3, U3 IR2104, U4 INA240A3D, U5 SN65HVD230, U6 STM32F405RGTx, U9 INA240A1D, Y1 8MHz

Commit message: from PC
Parts:
- added C11: 15p, Capacitor_SMD:C_0603_1608Metric, F.Cu at (88.7, 97.0)
- added C12: 15p, Capacitor_SMD:C_0603_1608Metric, F.Cu at (88.7, 102.5)
- added C27: 100n, Capacitor_SMD:C_0504_1310Metric, F.Cu at (76.0, 104.0)
- added C8: 1u, Capacitor_SMD:C_0504_1310Metric, F.Cu at (81.0, 98.5)
Connections:
- J4 pad 1: SWDIO -> +3.3V
- J4 pad 2: GND -> SWDIO
- J4 pad 4: +3.3VA -> GND
- U5 pad 5: +3.3V -> unconnected-(U5-Vref-Pad5)
- U5 pad 8: unconnected-(U5-Rs-Pad8) -> Net-(U5-Rs)
- U6 pad 28: unconnected-(U6-PB2-Pad28) -> BOOT1
- U9 pad 1: GND -> Net-(U9--)
- U9 pad 3: unconnected-(U9-REF2-Pad3) -> /BLDC driver phase A/PWR_3.3V
- U9 pad 7: unconnected-(U9-REF1-Pad7) -> GND
- U9 pad 8: Net-(U3-COM) -> Net-(U9-+)
