File: PCB/BLDC_motor_driver/BLDC_motor_driver.kicad_pcb (KiCad board)
At the start: 2 copper layers, 11 parts, among them Q2 CSD18534Q5A, Q3 CSD18540Q5B, Q4 CSD18533Q5A, U1 INA240A1D, U2 AS5048A, U3 IR2104, U4 UCC27714D, U5 SN65HVD230, U6 STM32F405RGTx, U7 STM32F303K8Tx, U8 INA240A1D

Commit message: pcb progress
Parts:
- removed Q2: CSD18534Q5A, Package_TO_SOT_SMD:TDSON-8-1
- removed Q3: CSD18540Q5B, Package_TO_SOT_SMD:TDSON-8-1
- removed Q4: CSD18533Q5A, Package_TO_SOT_SMD:TDSON-8-1
- added Q8: CSD18533Q5A, Package_TO_SOT_SMD:TDSON-8-1, F.Cu at (115.9, 44.4)
- added Q9: CSD18533Q5A, Package_TO_SOT_SMD:TDSON-8-1, F.Cu at (115.9, 53.9)
- added U10: AS5048A, Package_SO:TSSOP-14_4.4x5mm_P0.65mm, F.Cu at (99.5, 109.0)
- added U9: INA240A1D, Package_SO:SOIC-8_3.9x4.9mm_P1.27mm, F.Cu at (105.5, 58.9)
- U1: value INA240A1D -> INA240A2D
- U4: value UCC27714D -> INA240A3D; footprint Package_SO:SOIC-14_3.9x8.7mm_P1.27mm -> Package_SO:SOIC-8_3.9x4.9mm_P1.27mm
- U8: value INA240A1D -> SN65HVD230
- moved U8 67.4 mm to (150.5, 85.9)
- moved U6 65.6 mm to (113.5, 108.5), turned to 90 degrees
- moved U7 61.3 mm to (137.3, 86.5)
- moved U2 52.8 mm to (137.0, 98.5), turned to 90 degrees
- moved U1 38.8 mm to (113.5, 71.6)
- moved U3 25.1 mm to (97.0, 51.1)
- moved U4 23.3 mm to (101.0, 71.0)
- moved U5 20.4 mm to (111.5, 95.5), turned to 90 degrees
Connections:
- U2 pad 1: unconnected-(U2-~{CSn}-Pad1) -> STM1_SPI1_CS
- U2 pad 2: unconnected-(U2-CLK-Pad2) -> STM1_SPI1_SCK
- U2 pad 3: unconnected-(U2-MISO-Pad3) -> STM1_SPI1_MISO
- U2 pad 4: unconnected-(U2-MOSI-Pad4) -> STM1_SPI1_MOSI
- U3 pad 1: unconnected-(U3-VCC-Pad1) -> /BLDC driver phase A/PWR_12V
- U3 pad 2: unconnected-(U3-IN-Pad2) -> /BLDC driver phase A/PWM_IN_A
- U3 pad 3: unconnected-(U3-~{SD}-Pad3) -> /BLDC driver phase A/SD_A
- U3 pad 4: unconnected-(U3-COM-Pad4) -> Net-(U3-COM)
- U3 pad 5: unconnected-(U3-LO-Pad5) -> Net-(U3-LO)
- U3 pad 6: unconnected-(U3-VS-Pad6) -> /BLDC driver phase A/PHASE A
- U3 pad 7: unconnected-(U3-HO-Pad7) -> Net-(U3-HO)
- U3 pad 8: unconnected-(U3-VB-Pad8) -> Net-(U3-VB)
- U4 pad 2: unconnected-(U4-LI-Pad2) -> Net-(U4-GND-Pad2)
- U4 pad 4: unconnected-(U4-EN/NC-Pad4) -> Net-(U4-GND-Pad2)
- U5 pad 1: unconnected-(U5-D-Pad1) -> STM2_CAN_TX
- U5 pad 4: unconnected-(U5-R-Pad4) -> STM2_CAN_RX
- U6 pad 21: unconnected-(U6-PA5-Pad21) -> STM2_SPI1_SCK
- U6 pad 22: unconnected-(U6-PA6-Pad22) -> STM2_SPI1_MISO
- U6 pad 23: unconnected-(U6-PA7-Pad23) -> STM2_SPI1_MOSI
- U6 pad 24: unconnected-(U6-PC4-Pad24) -> STM2_SPI1_CS
- U6 pad 44: unconnected-(U6-PA11-Pad44) -> STM2_CAN_RX
- U6 pad 45: unconnected-(U6-PA12-Pad45) -> STM2_CAN_TX
- U7 pad 11: unconnected-(U7-PA5-Pad11) -> STM1_SPI1_SCK
- U7 pad 12: unconnected-(U7-PA6-Pad12) -> STM1_SPI1_MISO
- U7 pad 13: unconnected-(U7-PA7-Pad13) -> STM1_SPI1_MOSI
- U7 pad 18: unconnected-(U7-PA8-Pad18) -> STM1_SPI1_CS
- U7 pad 21: unconnected-(U7-PA11-Pad21) -> STM1_CAN_RX
- U7 pad 22: unconnected-(U7-PA12-Pad22) -> STM1_CAN_TX
- U8 pad 1: unconnected-(U8---Pad1) -> STM1_CAN_TX
- U8 pad 2: Net-(U8-GND-Pad2) -> unconnected-(U8-GND-Pad2)
- U8 pad 4: Net-(U8-GND-Pad2) -> STM1_CAN_RX
Other:
- copper layers 2 -> 4

Commit message: updated schematic
Parts:
- added Y1: Crystal_GND24, Crystal:Crystal_SMD_EuroQuartz_MJ-4Pin_5.0x3.2mm, F.Cu at (70.3, 107.0)
- added Y2: Crystal, Crystal:Crystal_SMD_TXC_7A-2Pin_5x3.2mm, F.Cu at (85.0, 108.0)
- U10: moved to B.Cu
- moved U1 44.3 mm to (74.0, 91.6)
- moved U4 41.0 mm to (65.7, 91.8)
- moved U5 34.1 mm to (85.0, 117.0), turned to 180 degrees
- moved U8 33.6 mm to (120.8, 101.5), turned to 180 degrees
- moved Q8 26.9 mm to (94.0, 60.0), turned to 90 degrees
- moved U3 19.1 mm to (94.0, 70.0), turned to 90 degrees
- moved U6 15.9 mm to (99.0, 115.0), turned to 180 degrees
- moved U7 15.4 mm to (134.6, 101.7), turned to 180 degrees
- moved Q9 15.2 mm to (102.0, 60.0), turned to 90 degrees
- moved U10 14.0 mm to (100.0, 95.0), turned to 90 degrees
- moved U2 11.8 mm to (134.3, 87.0), turned to -90 degrees
- moved U9 11.7 mm to (102.0, 70.0), turned to 90 degrees
Connections:
- net PWR_3.3V renamed /BLDC driver phase A/PWR_3.3V
Other:
- board outline added: 100 x 100 mm

Commit message: updated schematic
Parts:
- removed Y2: Crystal, Crystal:Crystal_SMD_TXC_7A-2Pin_5x3.2mm
- added C10: 15p, Capacitor_SMD:C_0603_1608Metric, F.Cu at (110.5, 123.5)
- added C3: 10u, Capacitor_SMD:C_0504_1310Metric, F.Cu at (66.5, 112.9)
- added C4: 10u, Capacitor_SMD:C_0504_1310Metric, F.Cu at (80.0, 105.0)
- added C5: 100n, Capacitor_SMD:C_0504_1310Metric, F.Cu at (66.5, 115.5)
- added C6: 100n, Capacitor_SMD:C_0504_1310Metric, F.Cu at (80.0, 107.6)
- added C9: 15p, Capacitor_SMD:C_0603_1608Metric, F.Cu at (110.5, 115.0)
- added J2: Screw_Terminal_01x02, TerminalBlock:TerminalBlock_Xinya_XY308-2.54-2P_1x02_P2.54mm_Horizontal, F.Cu at (72.0, 126.0)
- added J3: Conn_01x04_Socket, Connector_PinHeader_2.54mm:PinHeader_1x04_P2.54mm_Vertical, F.Cu at (84.0, 127.9)
- added R6: 120R, Resistor_SMD:R_0402_1005Metric, F.Cu at (69.5, 112.5)
- Y1: value Crystal_GND24 -> 8MHz
- moved Y1 41.8 mm to (110.3, 119.2), turned to 90 degrees
Connections:
- U10 pad 10: unconnected-(U10-TEST-Pad10) -> GND
- U10 pad 11: unconnected-(U10-VDD5V-Pad11) -> +3.3V
- U10 pad 12: unconnected-(U10-VDD3V-Pad12) -> +3.3V
- U10 pad 13: unconnected-(U10-GND-Pad13) -> GND
- U10 pad 5: unconnected-(U10-TEST-Pad5) -> GND
- U10 pad 6: unconnected-(U10-TEST-Pad6) -> GND
- U10 pad 7: unconnected-(U10-TEST-Pad7) -> GND
- U10 pad 8: unconnected-(U10-TEST-Pad8) -> GND
- U10 pad 9: unconnected-(U10-TEST-Pad9) -> GND
- U2 pad 10: unconnected-(U2-TEST-Pad10) -> GND
- U2 pad 11: unconnected-(U2-VDD5V-Pad11) -> +3.3V
- U2 pad 12: unconnected-(U2-VDD3V-Pad12) -> +3.3V
- U2 pad 13: unconnected-(U2-GND-Pad13) -> GND
- U2 pad 5: unconnected-(U2-TEST-Pad5) -> GND
- U2 pad 6: unconnected-(U2-TEST-Pad6) -> GND
- U2 pad 7: unconnected-(U2-TEST-Pad7) -> GND
- U2 pad 8: unconnected-(U2-TEST-Pad8) -> GND
- U2 pad 9: unconnected-(U2-TEST-Pad9) -> GND
- U5 pad 2: unconnected-(U5-GND-Pad2) -> GND
- U5 pad 3: unconnected-(U5-VCC-Pad3) -> +3.3V
- U5 pad 5: unconnected-(U5-Vref-Pad5) -> +3.3V
- U5 pad 6: unconnected-(U5-CANL-Pad6) -> Net-(J2-Pin_2)
- U5 pad 7: unconnected-(U5-CANH-Pad7) -> Net-(J2-Pin_1)
- U6 pad 1: unconnected-(U6-VBAT-Pad1) -> +3.3V
- U6 pad 12: unconnected-(U6-VSSA-Pad12) -> GND
- U6 pad 13: unconnected-(U6-VDDA-Pad13) -> +3.3VA
- U6 pad 18: Net-(U6-VSS-Pad18) -> GND
- U6 pad 19: unconnected-(U6-VDD-Pad19) -> +3.3V
- U6 pad 31: unconnected-(U6-VCAP_1-Pad31) -> Net-(U6-VCAP_1)
- U6 pad 32: unconnected-(U6-VDD-Pad32) -> +3.3V
- U6 pad 47: unconnected-(U6-VCAP_2-Pad47) -> Net-(U6-VCAP_2)
- U6 pad 48: unconnected-(U6-VDD-Pad48) -> +3.3V
- U6 pad 5: unconnected-(U6-PH0-Pad5) -> Net-(U6-PH0)
- U6 pad 6: unconnected-(U6-PH1-Pad6) -> Net-(U6-PH1)
- U6 pad 63: Net-(U6-VSS-Pad18) -> GND
- U6 pad 64: unconnected-(U6-VDD-Pad64) -> +3.3V
- U6 pad 7: unconnected-(U6-NRST-Pad7) -> Net-(U6-NRST)
- Y1 pad 1: unconnected-(Y1-Pad1) -> Net-(U6-PH0)
- Y1 pad 2: unconnected-(Y1-Pad2) -> GND
- Y1 pad 3: unconnected-(Y1-Pad3) -> Net-(U6-PH1)
- Y1 pad 4: unconnected-(Y1-Pad4) -> GND

Commit message: more pcb progress
Parts:
- removed C4: 10u, Capacitor_SMD:C_0504_1310Metric
- removed U2: AS5048A, Package_SO:TSSOP-14_4.4x5mm_P0.65mm
- removed U7: STM32F303K8Tx, Package_QFP:LQFP-32_7x7mm_P0.8mm
- removed U8: SN65HVD230, Package_SO:SOIC-8_3.9x4.9mm_P1.27mm
- added C7: 22u, Capacitor_SMD:C_0504_1310Metric, F.Cu at (124.0, 113.5)
- added D2: LED, LED_SMD:LED_0402_1005Metric, F.Cu at (120.5, 113.5)
- added H1: MountingHole, MountingHole:MountingHole_2.2mm_M2, F.Cu at (134.0, 68.0)
- added H2: MountingHole, MountingHole:MountingHole_2.2mm_M2, F.Cu at (65.0, 67.5)
- added H3: MountingHole, MountingHole:MountingHole_2.2mm_M2, F.Cu at (64.5, 121.5)
- added H4: MountingHole, MountingHole:MountingHole_2.2mm_M2, F.Cu at (136.0, 122.5)
- added J1: Current Sensing, TerminalBlock:TerminalBlock_Xinya_XY308-2.54-3P_1x03_P2.54mm_Horizontal, F.Cu at (134.9, 111.0)
- added J4: Conn_01x04_Socket, Connector_PinSocket_2.54mm:PinSocket_1x04_P2.54mm_Horizontal, F.Cu at (95.9, 134.5)
- added R7: 1k5, Resistor_SMD:R_0402_1005Metric, F.Cu at (122.5, 111.0)
- added U11: AMS1117-3.3, Package_TO_SOT_SMD:SOT-223-3_TabPin2, F.Cu at (122.0, 119.5)
- C6: value 100n -> 22u
- J2: value Screw_Terminal_01x02 -> CAN H/L
- J3: value Conn_01x04_Socket -> PWR; footprint Connector_PinHeader_2.54mm:PinHeader_1x04_P2.54mm_Vertical -> TerminalBlock:TerminalBlock_Xinya_XY308-2.54-2P_1x02_P2.54mm_Horizontal
- moved C6 51.0 mm to (128.5, 123.5)
- moved J3 38.0 mm to (122.0, 129.0)
- moved C3 15.9 mm to (82.3, 114.2), turned to 90 degrees
- moved R6 13.6 mm to (75.0, 125.0), turned to 180 degrees
- moved C5 12.9 mm to (79.3, 114.2), turned to 90 degrees
- moved J2 6.73 mm to (76.5, 131.0)
- moved U5 3.82 mm to (82.3, 119.7)
Connections:
- net STM2_CAN_RX renamed CAN_RX
- net STM2_CAN_TX renamed CAN_TX
- net STM2_SPI1_CS renamed SPI1_CS
- net STM2_SPI1_MISO renamed SPI1_MISO
- net STM2_SPI1_MOSI renamed SPI1_MOSI
- net STM2_SPI1_SCK renamed SPI1_SCK
- C6 pad 1: +3.3V -> +5V
- J3 pad 1: unconnected-(J3-Pin_1-Pad1) -> +5V
- J3 pad 2: unconnected-(J3-Pin_2-Pad2) -> GND
- U6 pad 46: unconnected-(U6-PA13-Pad46) -> SWDIO
- U6 pad 49: unconnected-(U6-PA14-Pad49) -> SWCLK
- U6 pad 60: unconnected-(U6-BOOT0-Pad60) -> BOOT0

Commit message: further PCB progress
Parts:
- added C13: C, Capacitor_SMD:C_0201_0603Metric, F.Cu at (112.7, 98.5)
- added C14: 100n, Capacitor_SMD:C_0201_0603Metric, F.Cu at (94.7, 102.5)
- added C15: 100n, Capacitor_SMD:C_0201_0603Metric, F.Cu at (101.7, 102.5)
- added C16: 100n, Capacitor_SMD:C_0201_0603Metric, F.Cu at (98.2, 102.5)
- added C17: 100n, Capacitor_SMD:C_0201_0603Metric, F.Cu at (104.8, 102.5)
- added C18: 10n, Capacitor_SMD:C_0201_0603Metric, F.Cu at (115.0, 104.5)
- added C19: 1u, Capacitor_SMD:C_0201_0603Metric, F.Cu at (118.2, 104.5)
- added C20: 4.7u, Capacitor_SMD:C_0201_0603Metric, F.Cu at (91.0, 102.5)
- added C21: 1u, Capacitor_SMD:C_0201_0603Metric, F.Cu at (121.2, 104.5)
- added C22: 100n, Capacitor_SMD:C_0201_0603Metric, F.Cu at (127.2, 105.0)
- added C23: 100n, Capacitor_SMD:C_0201_0603Metric, F.Cu at (131.2, 105.0)
- added C27: 100n, Capacitor_SMD:C_0504_1310Metric, F.Cu at (96.0, 130.5)
- added C28: 100n, Capacitor_SMD:C_0201_0603Metric, F.Cu at (107.8, 102.5)
- added C29: 100n, Capacitor_SMD:C_0504_1310Metric, F.Cu at (124.0, 115.0)
- added C4: 100n, Capacitor_SMD:C_0504_1310Metric, F.Cu at (127.0, 129.0)
- added C8: 1u, Capacitor_SMD:C_0504_1310Metric, F.Cu at (100.0, 87.5)
- added FB1: 120R, Inductor_SMD:L_Walsin_WLFM201209x, F.Cu at (107.0, 107.8)
- added J5: PHASE_A, TerminalBlock_MetzConnect:TerminalBlock_MetzConnect_360410_1x01_Horizontal_ScrewM3.0, F.Cu at (97.5, 49.5)
- added L2: L_Ferrite_Coupled_1324, Inductor_SMD:L_CommonModeChoke_Coilcraft_1812CAN, F.Cu at (75.2, 123.6)
- added R5: R, Resistor_SMD:R_0402_1005Metric, F.Cu at (107.5, 112.0)
- J2: value CAN H/L -> PWR
- J3: value PWR -> CAN H/L
- R7: value 1k5 -> 100R
- moved H4 90.4 mm to (68.0, 63.0)
- moved H3 89.3 mm to (132.0, 63.0)
- moved H2 59.6 mm to (68.0, 127.0)
- moved H1 59.0 mm to (132.0, 127.0)
- moved J3 46.1 mm to (76.0, 132.0)
- moved J2 44.0 mm to (120.5, 132.5), turned to 0 degrees
- moved C5 32.8 mm to (101.5, 90.0), turned to 0 degrees
- moved C3 29.1 mm to (98.5, 90.0), turned to 180 degrees
- moved J1 6.35 mm to (137.0, 117.0), turned to 90 degrees
- moved C7 4.50 mm to (124.0, 118.0)
- moved R7 4.03 mm to (120.5, 114.5), turned to 90 degrees
- moved D2 4.00 mm to (120.5, 117.5)
- moved U11 4.00 mm to (122.0, 123.5)
- moved R6 3.20 mm to (77.0, 127.5), turned to 0 degrees
- moved C6 2.50 mm to (127.0, 125.5)
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Connections:
- net /BLDC driver phase A/PHASE A renamed Net-(J5-Pin_1)
- J2 pad 1: Net-(J2-Pin_1) -> GND
- J2 pad 2: Net-(J2-Pin_2) -> +5V
- J3 pad 1: +5V -> Net-(J3-Pin_1)
- J3 pad 2: GND -> Net-(J3-Pin_2)
- J4 pad 1: SWDIO -> +3.3V
- J4 pad 2: GND -> SWDIO
- J4 pad 4: +3.3VA -> GND
- R6 pad 1: Net-(J2-Pin_1) -> Net-(J3-Pin_1)
- R6 pad 2: Net-(J2-Pin_2) -> Net-(J3-Pin_2)
- U5 pad 5: +3.3V -> unconnected-(U5-Vref-Pad5)
- U5 pad 6: Net-(J2-Pin_2) -> Net-(U5-CANL)
- U5 pad 7: Net-(J2-Pin_1) -> Net-(U5-CANH)
- U5 pad 8: unconnected-(U5-Rs-Pad8) -> Net-(U5-Rs)
- U6 pad 28: unconnected-(U6-PB2-Pad28) -> BOOT1
- U9 pad 1: GND -> Net-(U9--)
- U9 pad 3: unconnected-(U9-REF2-Pad3) -> /BLDC driver phase A/PWR_3.3V
- U9 pad 7: unconnected-(U9-REF1-Pad7) -> GND
- U9 pad 8: Net-(U3-COM) -> Net-(U9-+)

Commit message: PCB schematic progress - footprints and values
Parts:
- C13: value C -> 0.1u
- R5: value R -> 10k
Changed lines of the file:
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@@
 			)
 		)
-		(property "Value" "C"
+		(property "Value" "0.1u"
 			(at 0 1.05 0)
 			(layer "F.Fab")
@@
 			)
 		)
-		(property "Value" "R"
+		(property "Value" "10k"
 			(at 0 1.17 0)
 			(layer "F.Fab")

Commit message: PCB v2 progress...
Parts:
- removed C6, C7: 22u, Capacitor_SMD:C_0504_1310Metric
- removed J5: PHASE_A, TerminalBlock_MetzConnect:TerminalBlock_MetzConnect_360410_1x01_Horizontal_ScrewM3.0
- removed U9: INA240A1D, Package_SO:SOIC-8_3.9x4.9mm_P1.27mm
- added C1: 2.2u, Capacitor_Tantalum_SMD:CP_EIA-2012-12_Kemet-R, F.Cu at (95.0, 73.6)
- added C11: 100n, Capacitor_Tantalum_SMD:CP_EIA-2012-12_Kemet-R, F.Cu at (95.0, 83.4)
- added C12: 22u, Capacitor_Tantalum_SMD:CP_EIA-2012-12_Kemet-R, F.Cu at (61.6, 87.5)
- added C2: 470u, Capacitor_Tantalum_SMD:CP_EIA-2012-12_Kemet-R, F.Cu at (97.5, 82.4)
- added C24: 100n, Capacitor_SMD:C_0402_1005Metric, F.Cu at (86.9, 119.8)
- added C25: 100n, Capacitor_SMD:C_0402_1005Metric, F.Cu at (112.5, 73.0)
- added C26: 100n, Capacitor_SMD:C_0402_1005Metric, F.Cu at (111.0, 71.5)
- added D3: 1N4148W, Diode_SMD:D_SOD-123, F.Cu at (95.0, 78.5)
- added D4: 1N4148W, Diode_SMD:D_SOD-123, F.Cu at (97.0, 67.7)
- added D5: 1N4148W, Diode_SMD:D_SOD-123, F.Cu at (106.5, 67.5)
- added H5: 12V, MountingHole:MountingHole_2.2mm_M2_Pad_TopBottom, F.Cu at (58.5, 82.0)
- added H6: GND, MountingHole:MountingHole_2.2mm_M2_Pad_TopBottom, F.Cu at (58.5, 93.0)
- added H7: PHASE A, MountingHole:MountingHole_2.2mm_M2_Pad_TopBottom, F.Cu at (100.0, 50.0)
- added R1: 10R, Resistor_SMD:R_0603_1608Metric, F.Cu at (99.2, 67.4)
- added R10: 510R, Resistor_SMD:R_0603_1608Metric, F.Cu at (115.6, 83.5)
- added R11: 4.7K, Resistor_SMD:R_0603_1608Metric, F.Cu at (106.7, 83.5)
- added R2: 10R, Resistor_SMD:R_0603_1608Metric, F.Cu at (104.3, 67.5)
- added R3: 2mR, Resistor_SMD:R_2512_6332Metric, F.Cu at (111.5, 66.0)
- added R8: 0R, Resistor_SMD:R_0402_1005Metric, F.Cu at (79.5, 123.5)
- added R9: 330R, Resistor_SMD:R_0603_1608Metric, F.Cu at (112.1, 83.5)
- C10, C9: footprint Capacitor_SMD:C_0603_1608Metric -> Capacitor_SMD:C_0402_1005Metric
- C13, C14, C15, C16, C17, C18, C19, C20, C21, C22, C23, C28: footprint Capacitor_SMD:C_0201_0603Metric -> Capacitor_SMD:C_0402_1005Metric
- C27, C29, C3, C4, C5, C8: footprint Capacitor_SMD:C_0504_1310Metric -> Capacitor_SMD:C_0402_1005Metric
- U4: value INA240A3D -> LMV393; footprint Package_SO:SOIC-8_3.9x4.9mm_P1.27mm -> Package_SO:VSSOP-8_2.3x2mm_P0.5mm
- moved U4 51.0 mm to (114.2, 76.6), turned to 90 degrees
- moved U1 38.4 mm to (109.1, 76.0), turned to 90 degrees
- moved Q8 9.60 mm to (104.6, 60.6)
- moved U3 7.82 mm to (101.5, 75.0)
- moved Q9 5.41 mm to (97.6, 60.6)
- moved C4 4.98 mm to (122.0, 129.0), turned to 180 degrees
- moved J2 1.00 mm to (120.5, 133.5)
Connections:
- net Net-(J5-Pin_1) renamed /BLDC driver phase A/PHASE A
- Q8 pad 1: Net-(U3-COM) -> Net-(U1-+)
- Q8 pad 2: Net-(U3-COM) -> Net-(U1-+)
- Q8 pad 3: Net-(U3-COM) -> Net-(U1-+)
- Q9 pad 5: Net-(D1-K) -> /BLDC driver phase A/PWR_12V
- U1 pad 1: unconnected-(U1---Pad1) -> GND
- U1 pad 2: Net-(U1-GND-Pad2) -> GND
- U1 pad 3: unconnected-(U1-REF2-Pad3) -> GND
- U1 pad 4: Net-(U1-GND-Pad2) -> GND
- U1 pad 5: unconnected-(U1-Pad5) -> /BLDC driver phase A/VISENSE_A
- U1 pad 6: unconnected-(U1-V+-Pad6) -> /BLDC driver phase A/PWR_3.3V
- U1 pad 7: unconnected-(U1-REF1-Pad7) -> GND
- U1 pad 8: unconnected-(U1-+-Pad8) -> Net-(U1-+)
- U3 pad 3: /BLDC driver phase A/SD_A -> GND
- U3 pad 4: Net-(U3-COM) -> GND
- U4 pad 1: unconnected-(U4---Pad1) -> GND
- U4 pad 2: Net-(U4-GND-Pad2) -> Net-(U4A--)
- U4 pad 3: unconnected-(U4-REF2-Pad3) -> /BLDC driver phase A/VISENSE_A
- U4 pad 4: Net-(U4-GND-Pad2) -> (no net)
- U4 pad 5: unconnected-(U4-Pad5) -> (no net)
- U4 pad 6: unconnected-(U4-V+-Pad6) -> (no net)
- U4 pad 7: unconnected-(U4-REF1-Pad7) -> (no net)
- U4 pad 8: unconnected-(U4-+-Pad8) -> (no net)

Commit message: Test driver layour finished... final touches
Parts:
- moved C8 2.68 mm to (100.1, 90.2)
- moved C3 0.44 mm to (98.9, 90.2), turned to 90 degrees
- moved C5 0.27 mm to (101.3, 90.2), turned to 90 degrees
Changed lines of the file:
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@@
 	(footprint "Capacitor_SMD:C_0402_1005Metric"
 		(layer "F.Cu")
-		(at 101.5 90)
+		(at 101.3 90.18 90)
 		(descr "Capacitor SMD 0402 (1005 Metric), square (rectangular) end terminal, IPC-7351 nominal, (Body size source: IPC-SM-782 page 76, https://www.pcb-3d.com/wordpress/wp-content/uploads/ipc-sm-782a_amendment_1_and_2.pdf), generated with kicad-footprint-generator")
 		(tags "capacitor")
 		(property "Reference" "C5"
-			(at 0 -1.16 0)
+			(at 1.88 0.2 270)
 			(layer "F.SilkS")
 			(effects
@@
 		)
 		(property "Value" "100n"
-			(at 0 1.16 0)
+			(at 0.7 1.3 90)
 			(layer "F.Fab")
 			(effects
@@
 		)
 		(property "Datasheet" ""
-			(at 0 0 0)
+			(at 0 0 90)
 			(layer "F.Fab")
 			(hide yes)
@@
 		)
 		(property "Description" "Unpolarized capacitor"
-			(at 0 0 0)
+			(at 0 0 90)
 			(layer "F.Fab")
 			(hide yes)
@@
 		)
 		(fp_line
-			(start -0.91 -0.46)
-			(end 0.91 -0.46)
+			(start 0.91 -0.46)
+			(end 0.91 0.46)
 			(stroke
 				(width 0.05)
@@
 		)
 		(fp_line
-			(start -0.91 0.46)
-			(end -0.91 -0.46)
+			(start -0.91 -0.46)
+			(end 0.91 -0.46)
 			(stroke
 				(width 0.05)
@@
 		)
 		(fp_line
-			(start 0.91 -0.46)
-			(end 0.91 0.46)
+			(start 0.91 0.46)
+			(end -0.91 0.46)
 			(stroke
 				(width 0.05)
@@
 		)
 		(fp_line
-			(start 0.91 0.46)
-			(end -0.91 0.46)
+			(start -0.91 0.46)
+			(end -0.91 -0.46)
 			(stroke
 				(width 0.05)
@@
 		)
 		(fp_line
-			(start -0.5 -0.25)
-			(end 0.5 -0.25)
+			(start 0.5 -0.25)
+			(end 0.5 0.25)
 			(stroke
 				(width 0.1)
@@
 		)
 		(fp_line
-			(start -0.5 0.25)
-			(end -0.5 -0.25)
+			(start -0.5 -0.25)
+			(end 0.5 -0.25)
 			(stroke
 				(width 0.1)
@@
 		)
 		(fp_line
-			(start 0.5 -0.25)
-			(end 0.5 0.25)
+			(start 0.5 0.25)
+			(end -0.5 0.25)
 			(stroke
 				(width 0.1)
@@
 		)
 		(fp_line
-			(start 0.5 0.25)
-			(end -0.5 0.25)
+			(start -0.5 0.25)
+			(end -0.5 -0.25)
 			(stroke
 				(width 0.1)
@@
 		)
 		(fp_text user "${REFERENCE}"
-			(at 0 0 0)
+			(at 0 0 90)
 			(layer "F.Fab")
 			(effects
@@
 		)
 		(pad "1" smd roundrect
-			(at -0.48 0)
+			(at -0.48 0 90)
 			(size 0.56 0.62)
 			(layers "F.Cu" "F.Mask" "F.Paste")
@@
 		)
 		(pad "2" smd roundrect
-			(at 0.48 0)
+			(at 0.48 0 90)
 			(size 0.56 0.62)
 			(layers "F.Cu" "F.Mask" "F.Paste")
@@
 	(footprint "Capacitor_SMD:C_0402_1005Metric"
 		(layer "F.Cu")
-		(at 99.96 87.5 90)
+		(at 100.1 90.18 90)
 		(descr "Capacitor SMD 0402 (1005 Metric), square (rectangular) end terminal, IPC-7351 nominal, (Body size source: IPC-SM-782 page 76, https://www.pcb-3d.com/wordpress/wp-content/uploads/ipc-sm-782a_amendment_1_and_2.pdf), generated with kicad-footprint-generator")
 		(tags "capacitor")
 		(property "Reference" "C8"
-			(at 0 -1.16 90)
+			(at 1.9 0.1 90)
 			(layer "F.SilkS")
 			(effects
@@
 		)
 		(property "Value" "1u"
-			(at 0 1.16 90)
+			(at 3.68 0 90)
 			(layer "F.Fab")
 			(effects
@@
 	(footprint "Capacitor_SMD:C_0402_1005Metric"
 		(layer "F.Cu")
-		(at 98.5 90 180)
+		(at 98.9 90.18 90)
 		(descr "Capacitor SMD 0402 (1005 Metric), square (rectangular) end terminal, IPC-7351 nominal, (Body size source: IPC-SM-782 page 76, https://www.pcb-3d.com/wordpress/wp-content/uploads/ipc-sm-782a_amendment_1_and_2.pdf), generated with kicad-footprint-generator")
 		(tags "capacitor")
 		(property "Reference" "C3"
-			(at 0 -1.16 180)
+			(at 1.88 0 90)
 			(layer "F.SilkS")
 			(effects
@@
 		)
 		(property "Value" "10u"
-			(at 0 1.16 180)
+			(at 0.3 -1.2 90)
 			(layer "F.Fab")
 			(effects
@@
 		)
 		(property "Datasheet" ""
-			(at 0 0 180)
+			(at 0 0 90)
 			(layer "F.Fab")
 			(hide yes)
@@
 		)
 		(property "Description" "Unpolarized capacitor"
-			(at 0 0 180)
+			(at 0 0 90)
 			(layer "F.Fab")
 			(hide yes)
@@
 		(attr smd)
 		(fp_line
-			(start -0.107836 0.36)
-			(end 0.107836 0.36)
+			(start -0.107836 -0.36)
+			(end 0.107836 -0.36)
 			(stroke
 				(width 0.12)
@@
 		)
 		(fp_line
-			(start -0.107836 -0.36)
-			(end 0.107836 -0.36)
+			(start -0.107836 0.36)
+			(end 0.107836 0.36)
 			(stroke
 				(width 0.12)
@@
 		)
 		(fp_line
-			(start 0.91 0.46)
-			(end -0.91 0.46)
+			(start 0.91 -0.46)
+			(end 0.91 0.46)
 			(stroke
 				(width 0.05)
@@
 		)
 		(fp_line
-			(start 0.91 -0.46)
-			(end 0.91 0.46)
+			(start -0.91 -0.46)
+			(end 0.91 -0.46)
 			(stroke
 				(width 0.05)
@@
 		)
 		(fp_line
-			(start -0.91 0.46)
-			(end -0.91 -0.46)
+			(start 0.91 0.46)
+			(end -0.91 0.46)
 			(stroke
 				(width 0.05)
@@
 		)
 		(fp_line
-			(start -0.91 -0.46)
-			(end 0.91 -0.46)
+			(start -0.91 0.46)
+			(end -0.91 -0.46)
 			(stroke
 				(width 0.05)
@@
 		)
 		(fp_line
-			(start 0.5 0.25)
-			(end -0.5 0.25)
+			(start 0.5 -0.25)
+			(end 0.5 0.25)
 			(stroke
 				(width 0.1)
@@
 		)
 		(fp_line
-			(start 0.5 -0.25)
-			(end 0.5 0.25)
+			(start -0.5 -0.25)
+			(end 0.5 -0.25)
 			(stroke
 				(width 0.1)
@@
 		)
 		(fp_line
-			(start -0.5 0.25)
-			(end -0.5 -0.25)
+			(start 0.5 0.25)
+			(end -0.5 0.25)
 			(stroke
 				(width 0.1)
@@
 		)
 		(fp_line
-			(start -0.5 -0.25)
-			(end 0.5 -0.25)
+			(start -0.5 0.25)
+			(end -0.5 -0.25)
 			(stroke
 				(width 0.1)
@@
 		)
 		(fp_text user "${REFERENCE}"
-			(at 0 0 180)
+			(at 0 0 90)
 			(layer "F.Fab")
 			(effects
@@
 		)
 		(pad "1" smd roundrect
-			(at -0.48 0 180)
+			(at -0.48 0 90)
 			(size 0.56 0.62)
 			(layers "F.Cu" "F.Mask" "F.Paste")
@@
 		)
 		(pad "2" smd roundrect
-			(at 0.48 0 180)
+			(at 0.48 0 90)
 			(size 0.56 0.62)
 			(layers "F.Cu" "F.Mask" "F.Paste")
@@
 	)
 	(gr_circle
+		(center 100 95)
+		(end 106 95)
+		(stroke
+			(width 0.1)
+			(type default)
+		)
+		(fill no)
+		(layer "B.SilkS")
+	)
+	(gr_circle
