File: PCB/BLDC_motor_driver_testing/BLDC_motor_driver_testing.kicad_pcb (KiCad board)
At the start: 2 copper layers, 80 x 80 mm, 20 parts, among them Q2 IRF540N, Q3 IRF540N, U2 IR2104, U9 INA240A1D

Commit message: further progress
Parts:
- removed R10, R4, R9: R, Resistor_SMD:R_0402_1005Metric
- added C3: 470u, Capacitor_SMD:CP_Elec_10x10, F.Cu at (44.7, 69.5)
- added U1: LMV393, Package_SO:VSSOP-8_2.3x2mm_P0.5mm, F.Cu at (58.6, 69.8)
- moved C1 5.47 mm to (56.6, 54.5), turned to 0 degrees
- moved R5 4.04 mm to (60.5, 53.5)
- moved Q2 4.02 mm to (57.4, 40.0)
- moved U2 3.74 mm to (52.9, 65.1)
- moved R1 3.52 mm to (57.0, 44.0)
- moved C2 2.80 mm to (66.5, 46.5), turned to -90 degrees
- moved D2 2.55 mm to (63.0, 43.0)
- moved C25 2.16 mm to (72.0, 66.3)
- moved R3 2.16 mm to (66.0, 56.3)
- moved U9 2.16 mm to (67.5, 66.2)
- moved C26 2.11 mm to (67.3, 62.5)
- moved Q3 1.52 mm to (57.5, 49.4)
Connections:
- C26 pad 1: Net-(U9-+) -> Net-(Q3-S)
- C26 pad 2: Net-(U9--) -> GND
- U9 pad 1: Net-(U9--) -> GND
- U9 pad 5: Net-(R4-Pad1) -> /BLDC driver phase A/VISENSE_A
- U9 pad 8: Net-(U9-+) -> Net-(Q3-S)

Commit message: PCB progress...
Parts:
- added C29: 100n, Capacitor_SMD:C_0504_1310Metric, F.Cu at (57.0, 82.0)
- added C4: 100n, Capacitor_SMD:C_0504_1310Metric, F.Cu at (57.0, 88.5)
- added D3: LED, LED_SMD:LED_0402_1005Metric, F.Cu at (57.0, 79.0)
- added J2: PWR, TerminalBlock:TerminalBlock_Xinya_XY308-2.54-2P_1x02_P2.54mm_Horizontal, F.Cu at (51.0, 94.5)
- added R6: 10R, Resistor_SMD:R_0402_1005Metric, F.Cu at (59.5, 74.5)
- added R7: 10R, Resistor_SMD:R_0402_1005Metric, F.Cu at (56.5, 74.5)
- added R8: 100R, Resistor_SMD:R_0402_1005Metric, F.Cu at (59.5, 79.0)
- added U11: AMS1117-3.3, Package_TO_SOT_SMD:SOT-223-3_TabPin2, F.Cu at (52.0, 85.2)
- C3: footprint Capacitor_SMD:CP_Elec_10x10 -> Capacitor_SMD:CP_Elec_8x10
- moved C3 5.22 mm to (49.0, 72.5)
Connections:
- net Net-(Q2-S) renamed /BLDC driver phase A/PHASE A
- U1 pad 1: unconnected-(U1-Pad1) -> /BLDC driver phase A/SD_IN
- U1 pad 2: unconnected-(U1A---Pad2) -> Net-(U1A--)
- U1 pad 3: unconnected-(U1A-+-Pad3) -> /BLDC driver phase A/VISENSE_A
- U2 pad 3: /BLDC driver phase A/SD_A -> /BLDC driver phase A/SD_IN
Routing:
- added copper zone on B.Cu, net /BLDC driver phase A/PHASE A
- added copper zone on F.Cu, net /BLDC driver phase A/PHASE A

Commit message: PCB progress...
Parts:
- added C11: 470u, Capacitor_SMD:CP_Elec_8x10, F.Cu at (132.0, 33.7)
- added C12: 2.2u, Capacitor_Tantalum_SMD:CP_EIA-3216-18_Kemet-A_HandSolder, F.Cu at (139.6, 40.2)
- added C13: 100n, Capacitor_Tantalum_SMD:CP_EIA-3216-12_Kemet-S_HandSolder, F.Cu at (139.6, 43.3)
- added C14: 100n, Capacitor_SMD:C_0805_2012Metric_Pad1.18x1.45mm_HandSolder, F.Cu at (141.6, 50.2)
- added C15: 100n, Capacitor_SMD:C_0805_2012Metric_Pad1.18x1.45mm_HandSolder, F.Cu at (141.6, 53.2)
- added C16: 470u, Capacitor_SMD:CP_Elec_8x10, F.Cu at (132.0, 64.3)
- added C17: 2.2u, Capacitor_Tantalum_SMD:CP_EIA-3216-18_Kemet-A_HandSolder, F.Cu at (139.6, 70.8)
- added C18: 100n, Capacitor_Tantalum_SMD:CP_EIA-3216-12_Kemet-S_HandSolder, F.Cu at (139.6, 74.0)
- added C19: 100n, Capacitor_SMD:C_0805_2012Metric_Pad1.18x1.45mm_HandSolder, F.Cu at (141.6, 80.8)
- added C2: 22u, Capacitor_SMD:C_0805_2012Metric_Pad1.18x1.45mm_HandSolder, F.Cu at (51.7, 97.1)
- added C20: 100n, Capacitor_SMD:C_0805_2012Metric_Pad1.18x1.45mm_HandSolder, F.Cu at (141.6, 83.8)
- added C3: 22u, Capacitor_SMD:C_0805_2012Metric_Pad1.18x1.45mm_HandSolder, F.Cu at (158.6, 72.8)
- added C4: 22u, Capacitor_SMD:C_0805_2012Metric_Pad1.18x1.45mm_HandSolder, F.Cu at (51.8, 90.1)
- added D10: 1N4148W, Diode_SMD:D_SOD-123, F.Cu at (133.6, 77.7)
- added D3: 1N4148W, Diode_SMD:D_SOD-123, F.Cu at (31.5, 33.5)
- added D4: 1N4148W, Diode_SMD:D_SOD-123, F.Cu at (31.5, 41.5)
- added D5: 1N4148W, Diode_SMD:D_SOD-123, F.Cu at (133.6, 40.3)
- added D6: 1N4148W, Diode_SMD:D_SOD-123, F.Cu at (133.6, 43.6)
- added D7: 1N4148W, Diode_SMD:D_SOD-123, F.Cu at (133.6, 47.0)
- added D8: 1N4148W, Diode_SMD:D_SOD-123, F.Cu at (133.6, 71.0)
- added D9: 1N4148W, Diode_SMD:D_SOD-123, F.Cu at (133.6, 74.3)
- added H5: 12V, MountingHole:MountingHole_2.2mm_M2_Pad_TopBottom, F.Cu at (96.0, 38.5)
- added H6: GND, MountingHole:MountingHole_2.2mm_M2_Pad_TopBottom, F.Cu at (96.0, 48.5)
- added H8: PHASE B, MountingHole:MountingHole_2.2mm_M2_Pad_TopBottom, F.Cu at (60.0, 25.0)
- added H9: PHASE C, MountingHole:MountingHole_2.2mm_M2_Pad_TopBottom, F.Cu at (80.0, 25.0)
- added J2: SD_IN, TerminalBlock:TerminalBlock_Xinya_XY308-2.54-3P_1x03_P2.54mm_Horizontal, F.Cu at (62.5, 94.0)
- added J3: PWM_IN, TerminalBlock:TerminalBlock_Xinya_XY308-2.54-3P_1x03_P2.54mm_Horizontal, F.Cu at (73.9, 94.0)
- added J4: IN_SENSE_ADC, TerminalBlock:TerminalBlock_Xinya_XY308-2.54-3P_1x03_P2.54mm_Horizontal, F.Cu at (84.9, 94.0)
- added Q3: IRF540N, Package_TO_SOT_THT:TO-220-3_Vertical, F.Cu at (57.5, 32.0)
- added Q4: IRF540N, Package_TO_SOT_THT:TO-220-3_Vertical, F.Cu at (57.5, 40.0)
- added Q5: IRF540N, Package_TO_SOT_THT:TO-220-3_Vertical, F.Cu at (77.5, 32.0)
- added Q6: IRF540N, Package_TO_SOT_THT:TO-220-3_Vertical, F.Cu at (77.9, 40.0)
- added R10: 1mR, Resistor_SMD:R_2512_6332Metric, F.Cu at (118.6, 55.0)
- added R11: 330R, Resistor_SMD:R_0805_2012Metric_Pad1.20x1.40mm_HandSolder, F.Cu at (128.3, 46.0)
- added R12: 510R, Resistor_SMD:R_0805_2012Metric_Pad1.20x1.40mm_HandSolder, F.Cu at (128.3, 48.9)
- added R13: 4.7K, Resistor_SMD:R_0805_2012Metric_Pad1.20x1.40mm_HandSolder, F.Cu at (128.3, 51.9)
- added R14: 10R, Resistor_SMD:R_0805_2012Metric_Pad1.20x1.40mm_HandSolder, F.Cu at (128.3, 70.8)
- added R15: 10R, Resistor_SMD:R_0805_2012Metric_Pad1.20x1.40mm_HandSolder, F.Cu at (128.3, 73.7)
- added R16: 1mR, Resistor_SMD:R_2512_6332Metric, F.Cu at (118.6, 85.6)
- added R17: 330R, Resistor_SMD:R_0805_2012Metric_Pad1.20x1.40mm_HandSolder, F.Cu at (128.3, 76.7)
- added R18: 510R, Resistor_SMD:R_0805_2012Metric_Pad1.20x1.40mm_HandSolder, F.Cu at (128.3, 79.6)
- added R19: 4.7K, Resistor_SMD:R_0805_2012Metric_Pad1.20x1.40mm_HandSolder, F.Cu at (128.3, 82.5)
- added R7: 4.7K, Resistor_SMD:R_0805_2012Metric_Pad1.20x1.40mm_HandSolder, F.Cu at (47.0, 74.7)
- added R8: 10R, Resistor_SMD:R_0805_2012Metric_Pad1.20x1.40mm_HandSolder, F.Cu at (128.3, 40.1)
- added R9: 10R, Resistor_SMD:R_0805_2012Metric_Pad1.20x1.40mm_HandSolder, F.Cu at (128.3, 43.0)
- added U10: LMV393, Package_SO:VSSOP-8_2.3x2mm_P0.5mm, F.Cu at (141.0, 67.2)
- added U3: INA240A2D, Package_SO:SOIC-8_3.9x4.9mm_P1.27mm, F.Cu at (50.0, 68.6)
- added U5: IR2104, Package_DIP:DIP-8_W7.62mm_Socket_LongPads, F.Cu at (56.2, 53.0)
- added U6: INA240A2D, Package_SO:SOIC-8_3.9x4.9mm_P1.27mm, F.Cu at (134.9, 52.0)
- added U7: LMV393, Package_SO:VSSOP-8_2.3x2mm_P0.5mm, F.Cu at (141.0, 36.5)
- added U8: IR2104, Package_DIP:DIP-8_W7.62mm_Socket_LongPads, F.Cu at (76.2, 53.0)
- C1: renamed from C4; footprint Capacitor_SMD:C_0504_1310Metric -> Capacitor_SMD:C_0805_2012Metric_Pad1.18x1.45mm_HandSolder
- C10: renamed from C25; footprint Capacitor_SMD:C_0402_1005Metric -> Capacitor_SMD:C_0805_2012Metric_Pad1.18x1.45mm_HandSolder
- C5: renamed from C29; footprint Capacitor_SMD:C_0504_1310Metric -> Capacitor_SMD:C_0805_2012Metric_Pad1.18x1.45mm_HandSolder
- C7: renamed from C1; footprint Capacitor_Tantalum_SMD:CP_EIA-2012-15_AVX-P -> Capacitor_Tantalum_SMD:CP_EIA-3216-18_Kemet-A_HandSolder
- C8: renamed from C2; value 10u -> 100n; footprint Capacitor_Tantalum_SMD:CP_EIA-2012-15_AVX-P -> Capacitor_Tantalum_SMD:CP_EIA-3216-12_Kemet-S_HandSolder
- C9: renamed from C26; footprint Capacitor_SMD:C_0402_1005Metric -> Capacitor_SMD:C_0805_2012Metric_Pad1.18x1.45mm_HandSolder
- D1: renamed from D3; footprint LED_SMD:LED_0402_1005Metric -> LED_SMD:LED_0805_2012Metric_Pad1.15x1.40mm_HandSolder
- R1: renamed from R8; footprint Resistor_SMD:R_0402_1005Metric -> Resistor_SMD:R_0805_2012Metric_Pad1.20x1.40mm_HandSolder
- R2: renamed from R1; footprint Resistor_SMD:R_0402_1005Metric -> Resistor_SMD:R_0805_2012Metric_Pad1.20x1.40mm_HandSolder
- R3: renamed from R5; footprint Resistor_SMD:R_0402_1005Metric -> Resistor_SMD:R_0805_2012Metric_Pad1.20x1.40mm_HandSolder
- R4: renamed from R3; value 2mR -> 1mR
- R5: renamed from R7; value 10R -> 330R; footprint Resistor_SMD:R_0402_1005Metric -> Resistor_SMD:R_0805_2012Metric_Pad1.20x1.40mm_HandSolder
- R6: value 10R -> 510R; footprint Resistor_SMD:R_0402_1005Metric -> Resistor_SMD:R_0805_2012Metric_Pad1.20x1.40mm_HandSolder
- U9: value INA240A1D -> INA240A2D
- moved U9 69.4 mm to (134.9, 82.7)
- moved D2 38.6 mm to (27.0, 57.0), turned to -90 degrees
- moved C7 31.2 mm to (25.5, 52.0)
- moved R6 25.1 mm to (35.0, 69.2)
- moved R2 22.4 mm to (36.5, 35.0), turned to 0 degrees
- moved Q2 22.1 mm to (37.5, 40.0)
- moved U4 21.5 mm to (37.6, 65.2), turned to 90 degrees
- moved Q1 21.5 mm to (37.5, 32.0)
- moved C6 21.4 mm to (28.0, 68.2)
- moved U2 20.7 mm to (36.2, 53.0)
- moved H7 20.0 mm to (40.0, 25.0)
- moved C8 19.8 mm to (47.0, 42.9)
- moved R5 17.8 mm to (39.5, 69.2)
- moved C9 17.0 mm to (50.5, 64.2)
- moved C10 16.6 mm to (55.5, 68.3)
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- renumbered C3 to C6, J2 to J1, Q2 to Q1, Q3 to Q2, U11 to U1, U1 to U4
Connections:
- net /BLDC driver phase A/PWR_12V renamed +12V
- C10 pad 1: /BLDC driver phase A/PWR_3.3V -> +3.3V
- C10 pad 2: GND -> SD_A
- C6 pad 2: GND -> SD_A
- C7 pad 1: Net-(U2-VB) -> Net-(D2-K)
- C8 pad 2: Net-(Q3-S) -> SD_A
- C9 pad 1: Net-(Q3-S) -> Net-(Q2-S)
- C9 pad 2: GND -> SD_A
- Q2 pad 3: Net-(Q3-S) -> Net-(Q2-S)
- R4 pad 1: Net-(Q3-S) -> Net-(Q2-S)
- R4 pad 2: GND -> SD_A
- R5 pad 2: /BLDC driver phase A/PWR_3.3V -> +3.3V
- R6 pad 1: GND -> SD_A
- U2 pad 2: /BLDC driver phase A/PWM_IN_A -> PWM_IN_A
- U2 pad 3: /BLDC driver phase A/SD_IN -> SD_A
- U2 pad 4: Net-(Q3-S) -> SD_A
- U2 pad 8: Net-(U2-VB) -> Net-(D2-K)
- U4 pad 1: /BLDC driver phase A/SD_IN -> SD_A
- U4 pad 3: /BLDC driver phase A/VISENSE_A -> IN_SENSE_A
- U9 pad 1: GND -> SD_C
- U9 pad 2: GND -> SD_C
- U9 pad 3: /BLDC driver phase A/PWR_3.3V -> SD_C
- U9 pad 4: GND -> SD_C
- U9 pad 5: /BLDC driver phase A/VISENSE_A -> IN_SENSE_C
- U9 pad 6: /BLDC driver phase A/PWR_3.3V -> +3.3V
- U9 pad 7: GND -> SD_C
- U9 pad 8: Net-(Q3-S) -> Net-(Q6-S)
Routing:
- removed copper zone on B.Cu, net /BLDC driver phase A/PHASE A
- removed copper zone on F.Cu, net /BLDC driver phase A/PHASE A

Commit message: PCB layouting...
Parts:
- moved C11 79.8 mm to (61.5, 71.0), turned to -90 degrees
- moved C8 72.2 mm to (-25.0, 37.0)
- moved C14 70.4 mm to (71.5, 57.0), turned to 180 degrees
- moved C3 68.7 mm to (96.0, 44.5)
- moved C15 65.6 mm to (76.5, 61.5), turned to 90 degrees
- moved U6 64.0 mm to (71.5, 61.0)
- moved R2 61.1 mm to (-24.0, 43.5), turned to 90 degrees
- moved D3 54.6 mm to (-23.0, 29.5)
- moved R10 52.6 mm to (67.0, 45.0), turned to -90 degrees
- moved D4 51.0 mm to (-19.5, 41.0)
- moved R16 49.7 mm to (90.0, 45.0), turned to -90 degrees
- moved C16 49.4 mm to (83.0, 70.5), turned to -90 degrees
- moved C7 48.9 mm to (-20.5, 35.4), turned to 90 degrees
- moved C19 25.9 mm to (118.5, 69.0), turned to 180 degrees
- moved R3 25.6 mm to (23.5, 51.5), turned to 90 degrees
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Connections:
- C10 pad 2: SD_A -> GND
- C11 pad 2: SD_B -> GND
- C13 pad 2: SD_B -> GND
- C14 pad 2: SD_B -> GND
- C15 pad 2: SD_B -> GND
- C16 pad 2: SD_C -> GND
- C18 pad 2: SD_C -> GND
- C19 pad 2: SD_C -> GND
- C20 pad 2: SD_C -> GND
- C6 pad 2: SD_A -> GND
- C8 pad 2: SD_A -> GND
- C9 pad 2: SD_A -> GND
- J2 pad 1: SD_C -> GND
- J2 pad 2: SD_B -> GND
- J2 pad 3: SD_A -> GND
- Q1 pad 2: Net-(D2-K) -> +12V
- Q3 pad 2: Net-(D5-K) -> +12V
- Q5 pad 2: Net-(D8-K) -> +12V
- R10 pad 2: SD_B -> GND
- R12 pad 1: SD_B -> GND
- R13 pad 1: SD_B -> GND
- R16 pad 2: SD_C -> GND
- R18 pad 1: SD_C -> GND
- R19 pad 1: SD_C -> GND
- R4 pad 2: SD_A -> GND
- R6 pad 1: SD_A -> GND
- R7 pad 1: SD_A -> GND
- U10 pad 1: SD_C -> GND
- U2 pad 3: SD_A -> GND
- U2 pad 4: SD_A -> GND
- U3 pad 1: SD_A -> GND
- U3 pad 2: SD_A -> GND
- U3 pad 3: SD_A -> GND
- U3 pad 4: SD_A -> GND
- U3 pad 7: SD_A -> GND
- U4 pad 1: SD_A -> GND
- U5 pad 3: SD_B -> GND
- U5 pad 4: SD_B -> GND
- U6 pad 1: SD_B -> GND
- U6 pad 2: SD_B -> GND
- U6 pad 3: SD_B -> GND
- U6 pad 4: SD_B -> GND
- U6 pad 7: SD_B -> GND
- U7 pad 1: SD_B -> GND
- U8 pad 3: SD_C -> GND
- U8 pad 4: SD_C -> GND
- U9 pad 1: SD_C -> GND
- U9 pad 2: SD_C -> GND
- U9 pad 3: SD_C -> GND
- U9 pad 4: SD_C -> GND
- U9 pad 7: SD_C -> GND

Commit message: PCB layout progress
Parts:
- moved R13 85.2 mm to (64.5, 73.0)
- moved U7 75.9 mm to (65.0, 67.5), turned to 90 degrees
- moved C12 73.1 mm to (50.0, 64.0), turned to 90 degrees
- moved R12 72.5 mm to (70.0, 67.5), turned to -90 degrees
- moved R11 69.2 mm to (70.0, 72.0), turned to -90 degrees
- moved C13 68.6 mm to (54.0, 74.4), turned to -90 degrees
- moved D5 66.3 mm to (50.0, 69.5), turned to -90 degrees
- moved C8 65.1 mm to (28.2, 74.5)
- moved D6 61.7 mm to (52.0, 55.1), turned to 90 degrees
- moved D4 57.0 mm to (35.7, 55.0)
- moved R8 55.7 mm to (54.5, 55.5), turned to 90 degrees
- moved R19 55.5 mm to (89.0, 73.0)
- moved D3 54.5 mm to (25.2, 54.8)
- moved R2 53.0 mm to (27.7, 55.1)
- moved C7 52.4 mm to (23.7, 63.5)
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Other:
- copper layers 2 -> 4

Commit message: Test driver layout progress...
Parts:
- moved C16 50.8 mm to (73.5, -8.50)
- moved C6 50.7 mm to (26.5, -8.50)
- moved C11 50.4 mm to (50.1, -8.50)
- moved C17 14.8 mm to (77.0, 51.0)
- moved D8 14.3 mm to (77.0, 57.0)
- moved C18 13.6 mm to (79.0, 61.0), turned to 0 degrees
- moved C8 13.6 mm to (27.0, 61.0), turned to 0 degrees
- moved C13 13.5 mm to (53.0, 61.0), turned to 0 degrees
- moved C12 13.0 mm to (51.0, 51.0)
- moved C7 12.6 mm to (25.0, 51.0)
- moved D5 12.5 mm to (51.0, 57.0)
- moved R15 12.5 mm to (88.0, 44.0)
- moved D2 12.3 mm to (25.0, 57.0)
- moved D10 12.2 mm to (91.0, 44.0)
- moved U8 12.1 mm to (80.0, 58.0)
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Other:
- board size 80 x 80 mm -> 90 x 80 mm

Commit message: Test driver layout...
Parts:
- moved C6 77.5 mm to (27.5, 69.0), turned to 0 degrees
- moved C2 8.00 mm to (51.7, 87.2)
- moved C4 8.00 mm to (51.8, 82.1)
- moved C5 8.00 mm to (51.7, 79.6)
- moved D1 8.00 mm to (50.7, 77.1)
- moved H3 8.00 mm to (25.0, 87.0)
- moved H4 8.00 mm to (105.0, 87.0)
- moved J1 8.00 mm to (35.0, 87.0)
- moved J2 8.00 mm to (63.0, 87.0)
- moved J3 8.00 mm to (73.0, 87.0)
- moved J4 8.00 mm to (83.0, 87.0)
- moved R1 8.00 mm to (55.3, 77.1)
- moved U1 8.00 mm to (45.8, 83.7)
- moved C1 7.75 mm to (51.7, 85.0)
- moved D10 2.24 mm to (89.0, 45.0)
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Connections:
- net Net-(Q2-S) renamed /BLDC driver phase A/GND_A
- net Net-(Q4-S) renamed /BLDC driver phase B/GND_B
- net Net-(Q6-S) renamed /BLDC driver phase C/GND_C
- J3 pad 1: PWM_IN_C -> PWM_IN_A
- J3 pad 3: PWM_IN_A -> PWM_IN_C
- J4 pad 1: IN_SENSE_C -> IN_SENSE_A
- J4 pad 3: IN_SENSE_A -> IN_SENSE_C
Routing:
- net +12V: track 0.00 -> 98.9 mm, vias 0 -> 150
- net GND: track 0.00 -> 58.3 mm
- net /BLDC driver phase B/PHASE B: track 0.00 -> 35.2 mm, vias 0 -> 46
- net /BLDC driver phase C/PHASE C: track 0.00 -> 28.5 mm, vias 0 -> 34
- net /BLDC driver phase A/PHASE A: track 0.00 -> 28.1 mm, vias 0 -> 34
- net /BLDC driver phase C/GND_C: track 0.00 -> 15.7 mm
- net /BLDC driver phase B/GND_B: track 0.00 -> 15.7 mm
- net /BLDC driver phase A/GND_A: track 0.00 -> 15.7 mm
- net Net-(D7-A): track 0.00 -> 12.6 mm
- net Net-(D6-A): track 0.00 -> 12.6 mm
- net Net-(D4-A): track 0.00 -> 12.6 mm
- net Net-(D3-A): track 0.00 -> 12.6 mm
- net Net-(D9-A): track 0.00 -> 12.6 mm
- net Net-(D10-A): track 0.00 -> 12.6 mm
- net +3.3V: track 0.00 -> 8.08 mm
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- added copper zone on B.Cu, net +12V
- added copper zone on F.Cu, net +12V
- added copper zone on In1.Cu, net +12V
- added copper zone on In2.Cu, net +12V
- added copper zone on F.Cu, net /BLDC driver phase A/GND_A
- added copper zone on B.Cu, net /BLDC driver phase A/PHASE A
- added copper zone on F.Cu, net /BLDC driver phase A/PHASE A
- added copper zone on In1.Cu, net /BLDC driver phase A/PHASE A
- added copper zone on In2.Cu, net /BLDC driver phase A/PHASE A
- added copper zone on F.Cu, net /BLDC driver phase B/GND_B
- added copper zone on B.Cu, net /BLDC driver phase B/PHASE B
- added copper zone on F.Cu, net /BLDC driver phase B/PHASE B
- added copper zone on In1.Cu, net /BLDC driver phase B/PHASE B
- added copper zone on In2.Cu, net /BLDC driver phase B/PHASE B
- added copper zone on F.Cu, net /BLDC driver phase C/GND_C
- added copper zone on B.Cu, net /BLDC driver phase C/PHASE C
- added copper zone on F.Cu, net /BLDC driver phase C/PHASE C
- added copper zone on In1.Cu, net /BLDC driver phase C/PHASE C
- added copper zone on In2.Cu, net /BLDC driver phase C/PHASE C

Commit message: Getting closer to finish ;)
Parts:
- J2: value SD_IN -> PHASE A
- J3: value PWM_IN -> PHASE B
- J4: value IN_SENSE_ADC -> PHASE C
- moved C16 76.6 mm to (77.5, 68.0)
- moved C11 76.5 mm to (51.5, 68.0)
- moved J1 71.3 mm to (104.5, 71.0), turned to 90 degrees
- moved C2 63.4 mm to (107.5, 57.0), turned to 90 degrees
- moved U1 62.9 mm to (105.0, 62.5), turned to 180 degrees
- moved C1 60.2 mm to (105.0, 57.0), turned to 90 degrees
- moved C4 56.1 mm to (102.0, 57.0), turned to 90 degrees
- moved C5 52.8 mm to (99.5, 57.0), turned to 90 degrees
- moved D1 50.9 mm to (99.0, 61.0), turned to 90 degrees
- moved R1 45.4 mm to (99.0, 65.0), turned to -90 degrees
- moved J2 29.2 mm to (35.9, 76.0)
- moved J3 14.9 mm to (62.4, 76.5)
- moved J4 11.7 mm to (86.9, 76.0)
- moved H3 9.00 mm to (25.0, 78.0)
- moved H4 9.00 mm to (105.0, 78.0)
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Connections:
- net IN_SENSE_C renamed ISENSE_C
- J2 pad 1: GND -> PWM_IN_A
- J2 pad 3: GND -> ISENSE_A
- J3 pad 1: PWM_IN_A -> PWM_IN_B
- J3 pad 2: PWM_IN_B -> GND
- J3 pad 3: PWM_IN_C -> ISENSE_B
- J4 pad 1: IN_SENSE_A -> PWM_IN_C
- J4 pad 2: IN_SENSE_B -> GND
- U3 pad 5: IN_SENSE_A -> ISENSE_A
- U4 pad 3: IN_SENSE_A -> ISENSE_A
- U6 pad 5: IN_SENSE_B -> ISENSE_B
- U7 pad 3: IN_SENSE_B -> ISENSE_B
Routing:
- net +3.3V: track 8.08 -> 61.8 mm
- net Net-(U4A--): track 0.00 -> 4.20 mm
- net Net-(U7A--): track 0.00 -> 4.20 mm
- net Net-(U10A--): track 0.00 -> 4.20 mm
- net ISENSE_A: track 0.00 -> 4.05 mm
- net ISENSE_C: track 0.00 -> 4.05 mm
- net ISENSE_B: track 0.00 -> 4.05 mm
- net GND: track 58.3 -> 61.7 mm
- net Net-(D1-K): track 0.00 -> 1.98 mm
- net +12V: vias 150 -> 142
- added copper zone on F.Cu, net +3.3V
- added copper zone on F.Cu, net +5V
- added copper zone on F.Cu, net GND
Other:
- board size 90 x 80 mm -> 90 x 63 mm
- board text added: "5V"
- board text added: "GND"
